Commit message: Snapshot in-progress workspace for isolated robot loading changes

File: src/robo_arch/robots/ur7e/assets/model.urdf (robot description, URDF)
Before this commit: robot ur7e, 12 links, 11 joints
Links:
- link base_link_inertia: geometry collision mesh filename=meshes/collision/base.obj; visual mesh filename=meshes/visual/base.obj
- link forearm_link: geometry collision mesh filename=meshes/collision/forearm.obj; visual mesh filename=meshes/visual/forearm.obj
- link shoulder_link: geometry collision mesh filename=meshes/collision/shoulder.obj; visual mesh filename=meshes/visual/shoulder.obj
- link upper_arm_link: geometry collision mesh filename=meshes/collision/upper_arm.obj; visual mesh filename=meshes/visual/upper_arm.obj
- link wrist_1_link: geometry collision mesh filename=meshes/collision/wrist_1.obj; visual mesh filename=meshes/visual/wrist_1.obj
- link wrist_2_link: geometry collision mesh filename=meshes/collision/wrist_2.obj; visual mesh filename=meshes/visual/wrist_2.obj
- link wrist_3_link: geometry collision mesh filename=meshes/collision/wrist_3.obj; visual mesh filename=meshes/visual/wrist_3.obj
